File: kbxLEDController-16ch.sch (KiCad schematic (older format))
At the start: 57 parts, among them J1 PWM_1-4, J2 PWM_5-8, J3 PWM_9-12, J4 PWM_13-16, J5 5 TO 24 VDC, J6 SERIAL+GPIO, Q1 PMV20ENR, Q10 PMV20ENR, Q11 PMV20ENR, Q12 PMV20ENR, Q13 PMV20ENR, Q14 PMV20ENR, Q15 PMV20ENR, Q16 PMV20ENR, Q2 PMV20ENR, Q3 PMV20ENR, Q4 PMV20ENR, Q5 PMV20ENR, Q6 PMV20ENR, Q7 PMV20ENR, Q8 PMV20ENR, Q9 PMV20ENR, SW1 RESET, SW2 BOOT/IO0, SW3 I34, SW4 I35, SW5 I36, SW6 I39, U1 ESP32-WROOM-32D, U2 AP2205-33Y, U3 TSOP382xx

Commit message: v3
Parts:
- added J7: PIR, Connector_PinSocket_2.54mm:PinSocket_1x03_P2.54mm_Vertical, symbol Connector_Generic:Conn_01x03
Connections:
- net GND: now also J7.3 (Pin_3)
- net GPIO2: now also J7.2 (Pin_2)
- net VDC: now also J7.1 (Pin_1)
Other:
- moved on the sheet: C8, U3
Changed lines of the file:
@@
 	1800 4750 1850 4750
 $Comp
-L power:GND #PWR048
+L power:GND #PWR049
 U 1 1 5F591505
 P 1550 7250
-F 0 "#PWR048" H 1550 7000 50  0001 C CNN
+F 0 "#PWR049" H 1550 7000 50  0001 C CNN
 F 1 "GND" H 1555 7077 50  0000 C CNN
 F 2 "" H 1550 7250 50  0001 C CNN
@@
 	6000 7450 6000 7400
 $Comp
-L power:GND #PWR053
+L power:GND #PWR055
 U 1 1 5F58EE2D
 P 6000 7450
-F 0 "#PWR053" H 6000 7200 50  0001 C CNN
+F 0 "#PWR055" H 6000 7200 50  0001 C CNN
 F 1 "GND" H 6000 7300 50  0000 C CNN
 F 2 "" H 6000 7450 50  0001 C CNN
@@
 	5750 7450 5750 7400
 $Comp
-L power:GND #PWR052
+L power:GND #PWR054
 U 1 1 5F58EE3A
 P 5750 7450
-F 0 "#PWR052" H 5750 7200 50  0001 C CNN
+F 0 "#PWR054" H 5750 7200 50  0001 C CNN
 F 1 "GND" H 5750 7300 50  0000 C CNN
 F 2 "" H 5750 7450 50  0001 C CNN
@@
 	5500 7450 5500 7400
 $Comp
-L power:GND #PWR051
+L power:GND #PWR053
 U 1 1 5F58EE47
 P 5500 7450
-F 0 "#PWR051" H 5500 7200 50  0001 C CNN
+F 0 "#PWR053" H 5500 7200 50  0001 C CNN
 F 1 "GND" H 5500 7300 50  0000 C CNN
 F 2 "" H 5500 7450 50  0001 C CNN
@@
 	5250 7450 5250 7400
 $Comp
-L power:GND #PWR050
+L power:GND #PWR052
 U 1 1 5F58EE54
 P 5250 7450
-F 0 "#PWR050" H 5250 7200 50  0001 C CNN
+F 0 "#PWR052" H 5250 7200 50  0001 C CNN
 F 1 "GND" H 5250 7300 50  0000 C CNN
 F 2 "" H 5250 7450 50  0001 C CNN
@@
 L Interface_Optical:TSOP382xx U3
 U 1 1 5FD3483F
-P 3650 6500
-F 0 "U3" V 3592 6788 50  0000 L CNN
-F 1 "TSOP382xx" V 3683 6788 50  0000 L CNN
-F 2 "OptoDevice:Vishay_MINICAST-3Pin" H 3600 6125 50  0001 C CNN
-F 3 "http://www.vishay.com/docs/82491/tsop382.pdf" H 4300 6800 50  0001 C CNN
-	1    3650 6500
+P 3750 6500
+F 0 "U3" V 3692 6788 50  0000 L CNN
+F 1 "TSOP382xx" V 3783 6788 50  0000 L CNN
+F 2 "OptoDevice:Vishay_MINICAST-3Pin" H 3700 6125 50  0001 C CNN
+F 3 "http://www.vishay.com/docs/82491/tsop382.pdf" H 4400 6800 50  0001 C CNN
+	1    3750 6500
 	0    1    1    0
 $EndComp
@@
 L power:GND #PWR046
 U 1 1 5FD38B42
-P 3450 6900
-F 0 "#PWR046" H 3450 6650 50  0001 C CNN
-F 1 "GND" H 3455 6727 50  0000 C CNN
-F 2 "" H 3450 6900 50  0001 C CNN
-F 3 "" H 3450 6900 50  0001 C CNN
-	1    3450 6900
+P 3550 6900
+F 0 "#PWR046" H 3550 6650 50  0001 C CNN
+F 1 "GND" H 3555 6727 50  0000 C CNN
+F 2 "" H 3550 6900 50  0001 C CNN
+F 3 "" H 3550 6900 50  0001 C CNN
+	1    3550 6900
 	1    0    0    -1
 $EndComp
@@
 L power:+3.3V #PWR045
 U 1 1 5FD39214
-P 4100 6850
-F 0 "#PWR045" H 4100 6700 50  0001 C CNN
-F 1 "+3.3V" H 4115 7023 50  0000 C CNN
-F 2 "" H 4100 6850 50  0001 C CNN
-F 3 "" H 4100 6850 50  0001 C CNN
-	1    4100 6850
-	1    0    0    -1
-$EndComp
-Wire Wire Line
-	4100 6850 4100 6950
-Wire Wire Line
-	4100 6950 3850 6950
-Wire Wire Line
-	3850 6950 3850 6900
-Text Label 3650 7150 1    50   ~ 0
+P 4200 6850
+F 0 "#PWR045" H 4200 6700 50  0001 C CNN
+F 1 "+3.3V" H 4215 7023 50  0000 C CNN
+F 2 "" H 4200 6850 50  0001 C CNN
+F 3 "" H 4200 6850 50  0001 C CNN
+	1    4200 6850
+	1    0    0    -1
+$EndComp
+Wire Wire Line
+	4200 6850 4200 6950
+Wire Wire Line
+	4200 6950 3950 6950
+Wire Wire Line
+	3950 6950 3950 6900
+Text Label 3750 7150 1    50   ~ 0
 GPI36
 Wire Wire Line
-	3650 6900 3650 7150
+	3750 6900 3750 7150
 $Comp
 L power:VDC #PWR027
@@
 	1    0    0    -1
 $EndComp
-Text Notes 3300 7600 0    100  ~ 0
+Text Notes 3400 7600 0    100  ~ 0
 IR Receiver
 Text Notes 7100 3900 0    100  ~ 0
@@
 L Device:C C8
 U 1 1 5FF71EDF
-P 3850 7100
-F 0 "C8" H 3965 7146 50  0000 L CNN
-F 1 "100 nF" H 3965 7055 50  0000 L CNN
-F 2 "Capacitor_SMD:C_0805_2012Metric" H 3888 6950 50  0001 C CNN
-F 3 "~" H 3850 7100 50  0001 C CNN
-F 4 "CC0805KRX7R7BB104" H 3850 7100 50  0001 C CNN "Part"
-	1    3850 7100
-	1    0    0    -1
-$EndComp
-Connection ~ 3850 6950
-$Comp
-L power:GND #PWR049
+P 3950 7100
+F 0 "C8" H 4065 7146 50  0000 L CNN
+F 1 "100 nF" H 4065 7055 50  0000 L CNN
+F 2 "Capacitor_SMD:C_0805_2012Metric" H 3988 6950 50  0001 C CNN
+F 3 "~" H 3950 7100 50  0001 C CNN
+F 4 "CC0805KRX7R7BB104" H 3950 7100 50  0001 C CNN "Part"
+	1    3950 7100
+	1    0    0    -1
+$EndComp
+Connection ~ 3950 6950
+$Comp
+L power:GND #PWR051
 U 1 1 5FF74947
-P 3850 7250
-F 0 "#PWR049" H 3850 7000 50  0001 C CNN
-F 1 "GND" H 3855 7077 50  0000 C CNN
-F 2 "" H 3850 7250 50  0001 C CNN
-F 3 "" H 3850 7250 50  0001 C CNN
-	1    3850 7250
+P 3950 7250
+F 0 "#PWR051" H 3950 7000 50  0001 C CNN
+F 1 "GND" H 3955 7077 50  0000 C CNN
+F 2 "" H 3950 7250 50  0001 C CNN
+F 3 "" H 3950 7250 50  0001 C CNN
+	1    3950 7250
 	1    0    0    -1
 $EndComp
@@
 Wire Wire Line
 	4900 5500 4900 5400
+$Comp
+L Connector_Generic:Conn_01x03 J7
+U 1 1 5FD36529
+P 2750 7150
+F 0 "J7" H 2830 7192 50  0000 L CNN
+F 1 "PIR" H 2830 7101 50  0000 L CNN
+F 2 "Connector_PinSocket_2.54mm:PinSocket_1x03_P2.54mm_Vertical" H 2750 7150 50  0001 C CNN
+F 3 "~" H 2750 7150 50  0001 C CNN
+	1    2750 7150
+	1    0    0    -1
+$EndComp
+$Comp
+L power:GND #PWR050
+U 1 1 5FD36DAC
+P 2550 7250
+F 0 "#PWR050" H 2550 7000 50  0001 C CNN
+F 1 "GND" H 2555 7077 50  0000 C CNN
+F 2 "" H 2550 7250 50  0001 C CNN
+F 3 "" H 2550 7250 50  0001 C CNN
+	1    2550 7250
+	1    0    0    -1
+$EndComp
+Text Label 2350 7150 0    50   ~ 0
+GPIO2
+Wire Wire Line
+	2550 7150 2350 7150
+$Comp
+L power:VDC #PWR048
+U 1 1 5FD4098A
+P 2550 7050
+F 0 "#PWR048" H 2550 6950 50  0001 C CNN
+F 1 "VDC" H 2565 7223 50  0000 C CNN
+F 2 "" H 2550 7050 50  0001 C CNN
+F 3 "" H 2550 7050 50  0001 C CNN
+	1    2550 7050
+	1    0    0    -1
+$EndComp
 $EndSCHEMATC
